Commit message: simulation updated

File: pndbt_description/urdf/pndbt.control.urdf.xacro (robot description, xacro)
@@ -1,20 +1,29 @@
 <?xml version="1.0" encoding="utf-8"?>
-	<robot name="bldc_sim" xmlns:xacro="http://ros.org/wiki/xacro">
+	<robot name="pndbt" xmlns:xacro="http://ros.org/wiki/xacro">
 	<xacro:include filename="$(find pndbt_description)/urdf/pndbt.urdf.xacro"/>
-			<transmission name="tran0">
-		     <type>transmission_interface/SimpleTransmission</type>
-		     <joint name="stand_rotor">
-		      <hardwareInterface>hardware_interface/EffortJointInterface</hardwareInterface>
-		     </joint>
-		     <actuator name="motor0">
-		      <hardwareInterface>hardware_interface/EffortJointInterface</hardwareInterface>
-		      <!--hardware_interface/-->
-		      <mechanicalReduction>6</mechanicalReduction>
-		     </actuator>
-		  	</transmission>
-		<gazebo>
-		  <plugin name="gazebo_ros_control" filename="libgazebo_ros_control.so">
-		    <robotNamespace>/bldc_sim</robotNamespace>
-		  </plugin>
-</gazebo>
+        <transmission name="shoulder_transmission">
+            <type>transmission_interface/SimpleTransmission</type>
+            <joint name="shoulder">
+                <hardwareInterface>hardware_interface/EffortJointInterface</hardwareInterface>
+            </joint>
+            <actuator name="shoulder_motor">
+                <hardwareInterface>EffortJointInterface</hardwareInterface>
+                <mechanicalReduction>1</mechanicalReduction>
+            </actuator>
+        </transmission>
+        <transmission name="elbow_transmission">
+            <type>transmission_interface/SimpleTransmission</type>
+            <joint name="elbow">
+                <hardwareInterface>hardware_interface/EffortJointInterface</hardwareInterface>
+            </joint>
+            <actuator name="elbow_motor">
+                <hardwareInterface>EffortJointInterface</hardwareInterface>
+                <mechanicalReduction>1</mechanicalReduction>
+            </actuator>
+        </transmission>
+    <gazebo>
+        <plugin filename="libgazebo_ros_control.so" name="ros_control">
+            <robotNamespace>/pndbt</robotNamespace>
+        </plugin>
+    </gazebo>
 </robot>

File: pndbt_description/urdf/pndbt.urdf.xacro (robot description, xacro)
@@ -1,10 +1,4 @@
 <?xml version="1.0" encoding="utf-8"?>
-	<robot name="bldc_sim" xmlns:xacro="http://ros.org/wiki/xacro">
-		<xacro:arg name="hardware_interface" default="PositionJointInterface"/>
-		<xacro:arg name="robot_name" default="bldc_sim"/>
-	  	<!-- Import all Gazebo-customization elements, including Gazebo colors -->
-  		<!-- <xacro:include filename="$(find pndbt_description)/urdf/pndbt.gazebo.xacro" />  -->
-  		<!-- Import Transmissions -->
- 		<!-- <xacro:include filename="$(find pndbt_description)/urdf/pndbt.transmission.xacro" /> -->
+	<robot name="pndbt" xmlns:xacro="http://ros.org/wiki/xacro">
 <!--SOME PROPERTIES!-->
 		<xacro:property name="table_length" value="3" />
@@ -57,151 +51,12 @@
 		</gazebo>
 		<link name ="world"/>
-<!--FLOOR!-->
-	 	<link name="table_down">
-	   		<visual>
-	    			<geometry>
-	        			<box size ="${2*table_width} ${2*table_length} ${table_height}"/>
-	    			</geometry>
-	    			<origin xyz ="0 0 ${table_height/2}"/>
-	    			<material name="blue">
-        				<color rgba="0 0 0.8 1"/>
-     	    			</material>
-	   		</visual>
-			<collision>
-				<geometry>
-					<!--<box size ="${body_width} ${body_length} ${body_height}"/>!-->			<box size ="${2*table_width} ${2*table_length} ${table_height}"/>
-			        </geometry>
-			</collision>
-			<inertial>
-				<mass value="100"/>
-				<inertia
-				      ixx="1.0" ixy="0.0" ixz="0.0"
-				      iyy="1.0" iyz="0.0"
-				      izz="1.0"/>
-			</inertial>
-	 	</link>
-	 	<joint name="world_table_down" type="fixed">
-	 		<parent link="world"/>
-	 		<child link="table_down"/>
-			<origin rpy="0 0 0" xyz="0 0 ${table_height}"/>
-	 	</joint>
-<!--Foot #1!-->
-			<link name="foot_1">
-			   <visual>
-			    <geometry>
-				<box size ="${foot_width} ${foot_length} ${foot_height}"/>
-			    </geometry>
-			    <origin rpy="0 0 0" xyz ="0 0 0"/>
-			    <material name="black">
-					<color rgba="0 0 0 1"/>
-		     	    </material>
-			   </visual>
-			   <collision>
-				<geometry>
-					<box size ="${foot_width} ${foot_length} ${foot_height}"/>
-			        </geometry>
-			   </collision>
-			   <inertial>
-				<mass value="10"/>
-				<inertia
-				      ixx="1.0" ixy="0.0" ixz="0.0"
-				      iyy="1.0" iyz="0.0"
-				      izz="1.0"/>
-			   </inertial>
-			 </link>
-			 <joint name="table__down_foot_1" type="fixed">
-			 	<parent link="table_down"/>
-			 	<child link="foot_1"/>
-				<origin rpy="0 0 0" xyz="-${table_width/2-foot_width} -${table_length/2-foot_length} ${foot_height/2}"/>
-			 </joint>
-<!--Foot #2!-->
-			<link name="foot_2">
-			   <visual>
-			    <geometry>
-				<box size ="${foot_width} ${foot_length} ${foot_height}"/>
-			    </geometry>
-			    <origin rpy="0 0 0" xyz ="0 0 0"/>
-			    <material name="black">
-					<color rgba="0 0 0 1"/>
-		     	    </material>
-			   </visual>
-			   <collision>
-				<geometry>
-					<box size ="${foot_width} ${foot_length} ${foot_height}"/>
-			        </geometry>
-			   </collision>
-			   <inertial>
-				<mass value="10"/>
-				<inertia
-				      ixx="1.0" ixy="0.0" ixz="0.0"
-				      iyy="1.0" iyz="0.0"
-				      izz="1.0"/>
-			   </inertial>
-			 </link>
-			 <joint name="table__down_foot_2" type="fixed">
-			 	<parent link="table_down"/>
-			 	<child link="foot_2"/>
-				<origin rpy="0 0 0" xyz="${table_width/2-foot_width} -${table_length/2-foot_length} ${foot_height/2}"/>
-			 </joint>
-<!--Foot #3!-->
-			<link name="foot_3">
-			   <visual>
-			    <geometry>
-				<box size ="${foot_width} ${foot_length} ${foot_height}"/>
-			    </geometry>
-			    <origin rpy="0 0 0" xyz ="0 0 0"/>
-			    <material name="black">
-					<color rgba="0 0 0 1"/>
-		     	    </material>
-			   </visual>
-			   <collision>
-				<geometry>
-					<box size ="${foot_width} ${foot_length} ${foot_height}"/>
-			        </geometry>
-			   </collision>
-			   <inertial>
-				<mass value="10"/>
-				<inertia
-				      ixx="1.0" ixy="0.0" ixz="0.0"
-				      iyy="1.0" iyz="0.0"
-				      izz="1.0"/>
-			   </inertial>
-			 </link>
-			 <joint name="table__down_foot_3" type="fixed">
-			 	<parent link="table_down"/>
-			 	<child link="foot_3"/>
-				<origin rpy="0 0 0" xyz="${table_width/2-foot_width} ${table_length/2-foot_length} ${foot_height/2}"/>
-			 </joint>
-<!--Foot #4!-->
-			<link name="foot_4">
-			   <visual>
-			    <geometry>
-				<box size ="${foot_width} ${foot_length} ${foot_height}"/>
-			    </geometry>
-			    <origin rpy="0 0 0" xyz ="0 0 0"/>
-			    <material name="black">
-					<color rgba="0 0 0 1"/>
-		     	    </material>
-			   </visual>
-			   <collision>
-				<geometry>
-					<box size ="${foot_width} ${foot_length} ${foot_height}"/>
-			        </geometry>
-			   </collision>
-			   <inertial>
-				<mass value="10"/>
-				<inertia
-				      ixx="1.0" ixy="0.0" ixz="0.0"
-				      iyy="1.0" iyz="0.0"
-				      izz="1.0"/>
-			   </inertial>
-			 </link>
-			 <joint name="table__down_foot_4" type="fixed">
-			 	<parent link="table_down"/>
-			 	<child link="foot_4"/>
-				<origin rpy="0 0 0" xyz="-${table_width/2-foot_width} ${table_length/2-foot_length} ${foot_height/2}"/>
-			 </joint>
-<!--Table!-->
-	 	<link name="table_upper">
+      <joint name="grounding" type="fixed">
+        <parent link="world"/>
+        <child link="table"/>
+        <origin
+          xyz="0 0 1"
+          rpy="0 0 0" />
+      </joint>
+	 	<link name="table">
 	   		<visual>
 	    			<geometry>
@@ -213,9 +68,4 @@
      	    			</material>
 	   		</visual>
-			<collision>
-				<geometry>
-					<!--<box size ="${body_width} ${body_length} ${body_height}"/>!-->			<box size ="${table_width} ${table_length} ${table_height}"/>
-			        </geometry>
-			</collision>
 			<inertial>
 				<mass value="100"/>
@@ -226,9 +76,4 @@
 			</inertial>
 	 	</link>
-	 	<joint name="world_table_upper" type="fixed">
-	 		<parent link="table_down"/>
-	 		<child link="table_upper"/>
-			<origin rpy="0 0 0" xyz="0 0 ${foot_height+table_height}"/>
-	 	</joint>
 <!--Stand!-->
 	 	<link name="stand">
@@ -242,9 +87,4 @@
      	    			</material>
 	   		</visual>
-			<collision>
-				<geometry>
-					<box size ="${stand_length} ${stand_width} ${stand_height}"/>
-			        </geometry>
-			</collision>
 			<inertial>
 				<mass value="100"/>
@@ -256,5 +96,5 @@
 	 	</link>
 	 	<joint name="table_upper_stand" type="fixed">
-	 		<parent link="table_upper"/>
+	 		<parent link="table"/>
 	 		<child link="stand"/>
 			<origin rpy="0 0 0" xyz="${table_width/2-stand_length/2} 0 0"/>
@@ -271,9 +111,4 @@
      	    			</material>
 	   		</visual>
-			<collision>
-				<geometry>
-					<cylinder length ="${rotor_length}" radius="${rotor_radius}"/>
-			        </geometry>
-			</collision>
 			<inertial>
 				<mass value="0.10"/>
@@ -284,11 +119,8 @@
 			</inertial>
 	 	</link>
-	 	<joint name="stand_rotor" type="continuous">
-			<axis xyz="1 0 0"/>
-			<!--<limit effort="1000.0" lower="-3.1416" upper="3.1416" velocity="0.5"/>!-->
+	 	<joint name="stand_rotor" type="fixed">
 		 	<parent link="stand"/>
 		 	<child link="rotor"/>
 			<origin rpy="0 0 0" xyz="${stand_length/2+rotor_length/2} 0 ${stand_height/2}"/>
-			<dynamics damping="0.7"/>
 	 	</joint>
 	 	<link name="link1">
@@ -302,9 +134,4 @@
      	    			</material>
 	   		</visual>
-			<collision>
-				<geometry>
-					<box size ="0 0 0"/>
-			        </geometry>
-			</collision>
 			<inertial>
 				<origin rpy="0 0 0" xyz ="0 0 0.043"/>
@@ -316,8 +143,11 @@
 			</inertial>
 	 	</link>
-	 	<joint name="rotor_link1" type="fixed">
+	 	<joint name="shoulder" type="continuous">
 		 	<parent link="rotor"/>
 		 	<child link="link1"/>
+		 	<axis xyz="1 0 0"/>
 			<origin rpy="0 0 0" xyz="${rotor_length/2+link1_height/2} 0 0"/>
+			<!--<limit effort="1000.0" lower="-3.1416" upper="3.1416" velocity="0.5"/>!-->
+			<dynamics damping="0.0"/>
 	 	</joint>
 	 	<link name="link2">
@@ -345,5 +175,5 @@
 				</inertial>
 	 	</link>
-	 	<joint name="link1_link2" type="continuous">
+	 	<joint name="elbow" type="continuous">
 			<axis xyz="1 0 0"/>
 			<!--<limit effort="1000.0" lower="-3.1416" upper="3.1416" velocity="0.5"/>!-->

Commit message: code updates

File: pndbt_description/urdf/pndbt.control.urdf.xacro (robot description, xacro)
@@ -4,5 +4,5 @@
         <transmission name="shoulder_transmission">
             <type>transmission_interface/SimpleTransmission</type>
-            <joint name="shoulder">
+            <joint name="j1_shoulder">
                 <hardwareInterface>hardware_interface/EffortJointInterface</hardwareInterface>
             </joint>
@@ -14,5 +14,5 @@
         <transmission name="elbow_transmission">
             <type>transmission_interface/SimpleTransmission</type>
-            <joint name="elbow">
+            <joint name="j2_elbow">
                 <hardwareInterface>hardware_interface/EffortJointInterface</hardwareInterface>
             </joint>

File: pndbt_description/urdf/pndbt.urdf.xacro (robot description, xacro)
@@ -5,7 +5,4 @@
 		<xacro:property name="table_width" value="1.5" />
 		<xacro:property name="table_height" value="0.05" />
-		<xacro:property name="foot_height" value="0.80" />
-		<xacro:property name="foot_width" value="0.07" />
-		<xacro:property name="foot_length" value="0.07" />
 		<xacro:property name="stand_height" value="0.2" />
 		<xacro:property name="stand_length" value="0.4" />
@@ -135,13 +132,13 @@
 	   		</visual>
 			<inertial>
-				<origin rpy="0 0 0" xyz ="0 0 0.043"/>
-				<mass value="0.2"/>
+				<origin rpy="0 0 0" xyz ="0 0 -0.043"/>
+				<mass value="1.085"/>
 				<inertia
 				      ixx="1.0" ixy="0.0" ixz="0.0"
 				      iyy="1.0" iyz="0.0"
-				      izz="1.0"/>
+				      izz="0.008"/>
 			</inertial>
 	 	</link>
-	 	<joint name="shoulder" type="continuous">
+	 	<joint name="j1_shoulder" type="continuous">
 		 	<parent link="rotor"/>
 		 	<child link="link1"/>
@@ -161,19 +158,14 @@
      	    			</material>
 	   		</visual>
-			<collision>
-				<geometry>
-					<box size ="${link2_height} ${link2_width} ${link2_length}"/>
-			        </geometry>
-			</collision>
 			<inertial>
-				<origin rpy="0 0 0" xyz ="0 0 0.095"/>
-				<mass value="0.2"/>
+				<origin rpy="0 0 0" xyz ="0 0 -0.095"/>
+				<mass value="0.26"/>
 				<inertia
 				      ixx="1" ixy="0.0" ixz="0.0"
 				      iyy="1" iyz="0.0"
-				      izz="1"/>
+				      izz="0.002"/>
 				</inertial>
 	 	</link>
-	 	<joint name="elbow" type="continuous">
+	 	<joint name="j2_elbow" type="continuous">
 			<axis xyz="1 0 0"/>
 			<!--<limit effort="1000.0" lower="-3.1416" upper="3.1416" velocity="0.5"/>!-->
