Commit message: bag current vs torque

File: pndbt_description/urdf/pndbt.urdf.xacro (robot description, xacro)
@@ -14,8 +14,8 @@
 		<xacro:property name="rotor_radius" value="0.05" />
 		<xacro:property name="link1_height" value="0.05" />
-		<xacro:property name="link1_length" value="0.4" />
+		<xacro:property name="link1_length" value="0.250" />
 		<xacro:property name="link1_width" value="0.10" />
 		<xacro:property name="link2_height" value="0.05" />
-		<xacro:property name="link2_length" value="0.3" />
+		<xacro:property name="link2_length" value="0.250" />
 		<xacro:property name="link2_width" value="0.10" />
 		<xacro:property name="links_offset" value="0.06" />
@@ -302,4 +302,5 @@
 			</collision>
 			<inertial>
+				<origin rpy="0 0 0" xyz ="0 0 0.043"/>
 				<mass value="0.2"/>
 				<inertia
@@ -330,4 +331,5 @@
 			</collision>
 			<inertial>
+				<origin rpy="0 0 0" xyz ="0 0 0.095"/>
 				<mass value="0.2"/>
 				<inertia

Commit message: sim update

File: pndbt_description/urdf/pndbt.urdf.xacro (robot description, xacro)
@@ -1,4 +1,10 @@
 <?xml version="1.0" encoding="utf-8"?>
 	<robot name="bldc_sim" xmlns:xacro="http://ros.org/wiki/xacro">
+		<xacro:arg name="hardware_interface" default="PositionJointInterface"/>
+		<xacro:arg name="robot_name" default="bldc_sim"/>
+	  	<!-- Import all Gazebo-customization elements, including Gazebo colors -->
+  		<!-- <xacro:include filename="$(find pndbt_description)/urdf/pndbt.gazebo.xacro" />  -->
+  		<!-- Import Transmissions -->
+ 		<!-- <xacro:include filename="$(find pndbt_description)/urdf/pndbt.transmission.xacro" /> -->
 <!--SOME PROPERTIES!-->
 		<xacro:property name="table_length" value="3" />
@@ -20,34 +26,34 @@
 		<xacro:property name="link2_width" value="0.10" />
 		<xacro:property name="links_offset" value="0.06" />
-		  <gazebo reference="table_down">
-		    <material>Gazebo/Grey</material>
-		  </gazebo>
-		  <gazebo reference="table_upper">
-		    <material>Gazebo/GreyTransparent</material>
-		  </gazebo>
-		  <gazebo reference="foot_1">
-		    <material>Gazebo/DarkGrey</material>
-		  </gazebo>
-		  <gazebo reference="foot_2">
-		    <material>Gazebo/DarkGrey</material>
-		  </gazebo>
-		  <gazebo reference="foot_3">
-		    <material>Gazebo/DarkGrey</material>
-		  </gazebo>
-		  <gazebo reference="foot_4">
-		    <material>Gazebo/DarkGrey</material>
-		  </gazebo>
-		  <gazebo reference="stand">
-		    <material>Gazebo/Black</material>
-		  </gazebo>
+		<gazebo reference="table_down">
+		  <material>Gazebo/Grey</material>
+		</gazebo>
+		<gazebo reference="table_upper">
+		  <material>Gazebo/GreyTransparent</material>
+		</gazebo>
+		<gazebo reference="foot_1">
+		  <material>Gazebo/DarkGrey</material>
+		</gazebo>
+		<gazebo reference="foot_2">
+		  <material>Gazebo/DarkGrey</material>
+		</gazebo>
+		<gazebo reference="foot_3">
+		  <material>Gazebo/DarkGrey</material>
+		</gazebo>
+		<gazebo reference="foot_4">
+		  <material>Gazebo/DarkGrey</material>
+		</gazebo>
+		<gazebo reference="stand">
+		  <material>Gazebo/Black</material>
+		</gazebo>
 		<gazebo reference="rotor">
-		    <material>Gazebo/Blue</material>
-		  </gazebo>
+		  <material>Gazebo/Blue</material>
+		</gazebo>
 		<gazebo reference="link1">
-		    <material>Gazebo/Yellow</material>
-		  </gazebo>
+		  <material>Gazebo/Yellow</material>
+		</gazebo>
 		<gazebo reference="link2">
-		    <material>Gazebo/Red</material>
-		  </gazebo>
+		  <material>Gazebo/Red</material>
+		</gazebo>
 		<link name ="world"/>
 <!--FLOOR!-->

Commit message: control code update

File: pndbt_description/urdf/pndbt.urdf.xacro (robot description, xacro)
@@ -22,16 +22,4 @@
 		<gazebo reference="table_upper">
 		  <material>Gazebo/GreyTransparent</material>
-		</gazebo>
-		<gazebo reference="foot_1">
-		  <material>Gazebo/DarkGrey</material>
-		</gazebo>
-		<gazebo reference="foot_2">
-		  <material>Gazebo/DarkGrey</material>
-		</gazebo>
-		<gazebo reference="foot_3">
-		  <material>Gazebo/DarkGrey</material>
-		</gazebo>
-		<gazebo reference="foot_4">
-		  <material>Gazebo/DarkGrey</material>
 		</gazebo>
 		<gazebo reference="stand">
@@ -144,5 +132,5 @@
 		 	<child link="link1"/>
 		 	<axis xyz="1 0 0"/>
-			<origin rpy="0 0 0" xyz="${rotor_length/2+link1_height/2} 0 0"/>
+			<origin rpy="1.5707 0 0" xyz="${rotor_length/2+link1_height/2} 0 0"/>
 			<!--<limit effort="1000.0" lower="-3.1416" upper="3.1416" velocity="0.5"/>!-->
 			<dynamics damping="0.0"/>

Commit message: point stabilization modified

File: pndbt_description/urdf/pndbt.urdf.xacro (robot description, xacro)
@@ -134,5 +134,5 @@
 			<origin rpy="1.5707 0 0" xyz="${rotor_length/2+link1_height/2} 0 0"/>
 			<!--<limit effort="1000.0" lower="-3.1416" upper="3.1416" velocity="0.5"/>!-->
-			<dynamics damping="0.0"/>
+			<dynamics damping="0.001"/>
 	 	</joint>
 	 	<link name="link2">
@@ -161,5 +161,5 @@
 		 	<child link="link2"/>
 			<origin xyz="${links_offset} 0 -${link1_length}"/>
-			<dynamics damping="0.0"/>
+			<dynamics damping="0.001"/>
 	 	</joint>
 </robot>

Commit message: new updates

File: pndbt_description/urdf/pndbt.urdf.xacro (robot description, xacro)
@@ -134,5 +134,5 @@
 			<origin rpy="1.5707 0 0" xyz="${rotor_length/2+link1_height/2} 0 0"/>
 			<!--<limit effort="1000.0" lower="-3.1416" upper="3.1416" velocity="0.5"/>!-->
-			<dynamics damping="0.001"/>
+			<dynamics damping="0.000"/>
 	 	</joint>
 	 	<link name="link2">
@@ -161,5 +161,5 @@
 		 	<child link="link2"/>
 			<origin xyz="${links_offset} 0 -${link1_length}"/>
-			<dynamics damping="0.001"/>
+			<dynamics damping="0.000"/>
 	 	</joint>
 </robot>
